File: hardware/relay_expander/current/pcb/main_board/relays.kicad_sch (KiCad schematic)
At the start: 82 parts, among them J10 Screw_Terminal_01x02, J11 Screw_Terminal_01x02, J4 Screw_Terminal_01x02, J5 Screw_Terminal_01x02, J6 Screw_Terminal_01x02, J7 Screw_Terminal_01x02, J8 Screw_Terminal_01x02, J9 Screw_Terminal_01x02, K1 SANYOU_SRD_Form_C, K2 SANYOU_SRD_Form_C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

Commit message: [ADD] lauout for relay expander pcb
Parts:
- D10, D11, D12, D15, D16, D4, D5, D6: value 1N4007 -> 1N4148; footprint (none) -> Diode_SMD:D_SOD-123
- J10, J11, J5, J6, J7, J9: footprint Project_Parts_Footprints_Lib:TerminalBlock_Phoenix_MPT-0,5-3-2.54_1x03_P2.54mm_Horizontal -> footprints:Terminal_block_1x3_2,54
- J4: footprint Project_Parts_Footprints_Lib:TerminalBlock_Phoenix_MPT-0,5-3-2.54_1x03_P2.54mm_Horizontal -> TerminalBlock:TerminalBlock_Xinya_XY308-2.54-3P_1x03_P2.54mm_Horizontal
- J8: value Screw_Terminal_01x02 -> Screw_Terminal_01x03; footprint Project_Parts_Footprints_Lib:TerminalBlock_Phoenix_MPT-0,5-3-2.54_1x03_P2.54mm_Horizontal -> footprints:Terminal_block_1x3_2,54
- K1, K2, K3, K4, K5, K6, K7, K8: value SANYOU_SRD_Form_C -> HF46F-12-HS1; footprint templates_lib_footprints:Songle_SMI-SL-A -> homeautomation_core:relay_HF46F; symbol Relay:SANYOU_SRD_Form_A -> homeautomation_core:Relay_HF46F_Form_A
- R11, R12, R13, R14, R15, R16, R17, R18, R19, R23, R24, R25, R26, R27, R28, R29, R30, R33, R34, R35, R36, R5, R6, R7: footprint (none) -> Resistor_SMD:R_1206_3216Metric_Pad1.30x1.75mm_HandSolder
Connections:
- net +12V: now also K1.2, K2.2, K3.2, K4.2, K5.2, K6.2, K7.2, K8.2; no longer K1.5, K2.5, K3.5, K4.5, K5.5, K6.5, K7.5, K8.5
- net at J5.3 (Pin_3), JP3.1 (A): now also K2.3; no longer K2.1
- net at D14.1 (K), D16.2 (A), Q8.1 (C): now also K8.1; no longer K8.2
- net at D12.2 (A), D9.1 (K), Q6.1 (C): now also K6.1; no longer K6.2
- net at D2.1 (K), D5.2 (A), Q2.1 (C): now also K2.1; no longer K2.2
- net at J5.2 (Pin_2): now also K2.4; no longer K2.3
- net at J7.2 (Pin_2): now also K4.4; no longer K4.3
- net at J7.3 (Pin_3), JP5.1 (A): now also K4.3; no longer K4.1
- net at J11.3 (Pin_3), JP9.1 (A): now also K8.3; no longer K8.1
- net at J8.2 (Pin_2): now also K5.4; no longer K5.3
- net at J8.3 (Pin_3), JP6.1 (A): now also K5.3; no longer K5.1
- net at D11.2 (A), D8.1 (K), Q5.1 (C): now also K5.1; no longer K5.2
- net at D1.1 (K), D4.2 (A), Q1.1 (C): now also K1.1; no longer K1.2
- net at D3.1 (K), D6.2 (A), Q3.1 (C): now also K3.1; no longer K3.2
- net at J6.3 (Pin_3), JP4.1 (A): now also K3.3; no longer K3.1
- net at J6.2 (Pin_2): now also K3.4; no longer K3.3
- net at J10.2 (Pin_2): now also K7.4; no longer K7.3
- net at J10.3 (Pin_3), JP8.1 (A): now also K7.3; no longer K7.1
- net at J11.2 (Pin_2): now also K8.4; no longer K8.3
- net at D13.1 (K), D15.2 (A), Q7.1 (C): now also K7.1; no longer K7.2
- net at D10.2 (A), D7.1 (K), Q4.1 (C): now also K4.1; no longer K4.2
- net at J9.3 (Pin_3), JP7.1 (A): now also K6.3; no longer K6.1
- net at J9.2 (Pin_2): now also K6.4; no longer K6.3
- net at J4.2 (Pin_2): now also K1.4; no longer K1.3
- net at J4.3 (Pin_3), JP2.1 (A): now also K1.3; no longer K1.1
