File: hardware/relay_expander/current/pcb/ui_board/ui_board.kicad_sch (KiCad schematic)
At the start: 36 parts, among them J1 Conn_01x20_Socket

Commit message: [ADD] ui_board finished setup]
Connections:
- net at J1.17 (Pin_17): now also D13.1 (K)
