File: hardware/relay_expander/current/pcb/ui_board/ui_board.kicad_pcb (KiCad board)
At the start: 2 copper layers, 84 x 26 mm, 36 parts, among them J1 Conn_01x20_Socket

Commit message: [FIX] move connector on ui board
Parts:
- moved J1 2.50 mm to (177.5, 99.0)
Routing:
- net Net-(D9-K): track 65.1 -> 61.5 mm
- net Net-(D16-K): track 14.0 -> 10.7 mm
- net Net-(D11-K): track 49.8 -> 46.7 mm
- net Net-(D13-K): track 34.5 -> 31.9 mm
- net Net-(D5-K): track 41.5 -> 38.9 mm, vias 1 -> 0
- net Net-(D7-K): track 24.2 -> 21.7 mm, vias 1 -> 0
- net Net-(D3-K): track 59.7 -> 57.2 mm, vias 1 -> 0
- net Net-(D15-K): track 19.6 -> 17.1 mm
- net Net-(D2-K): track 57.5 -> 55.1 mm
- net +12V: track 69.4 -> 67.2 mm, vias 1 -> 0
- net Net-(D4-K): track 42.0 -> 40.1 mm
- net Net-(D1-K): track 76.6 -> 78.4 mm
- net +3V3: track 72.2 -> 70.7 mm
- net Net-(D6-K): track 26.5 -> 25.1 mm
- net Net-(D14-K): track 33.1 -> 33.7 mm
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
Commit message: [FIX] problem with connector to expander board
Parts:
- J1: footprint Connector_PinSocket_1.27mm:PinSocket_2x10_P1.27mm_Vertical -> homeautomation_core:PinSocket_2x10_P1.27mm_Vertical_Bottom
Changed lines of the file:
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@@
 		)
 	)
-	(footprint "Connector_PinSocket_1.27mm:PinSocket_2x10_P1.27mm_Vertical"
+	(footprint "homeautomation_core:PinSocket_2x10_P1.27mm_Vertical_Bottom"
 		(locked yes)
 		(layer "B.Cu")
@@
 		(tags "Through hole socket strip THT 2x10 1.27mm double row")
 		(property "Reference" "J1"
-			(at 0 7.8575 0)
+			(at -0.34 7.65 0)
 			(layer "B.SilkS")
 			(effects
@@
 		)
 		(property "Value" "Conn_01x20_Socket"
-			(at 0 -7.8425 0)
+			(at 1.01 -8.66 0)
 			(layer "B.Fab")
 			(effects
@@
 		)
 		(property "Datasheet" ""
-			(at 0.635 5.7225 0)
+			(at 1.645 1.8925 0)
 			(layer "B.Fab")
 			(hide yes)
@@
 			)
 		)
-		(property "Description" "Generic connector, single row, 01x20, script generated"
-			(at 0.635 5.7225 0)
+		(property "Description" ""
+			(at 1.645 1.8925 0)
 			(layer "B.Fab")
 			(hide yes)
@@
 		)
 		(property "KiLib_Generator" "connector/pin_header_socket"
-			(at 0.635 5.7225 0)
+			(at 1.645 1.8925 0)
 			(layer "B.SilkS")
 			(hide yes)
@@
 		)
 		(fp_line
+			(start 0 -6.4025)
+			(end 0 6.4025)
+			(stroke
+				(width 0.1)
+				(type solid)
+			)
+			(layer "B.SilkS")
+		)
+		(fp_line
 			(start -0.32747 6.4175)
 			(end -0.125 6.4175)
@@
 		)
 		(fp_line
+			(start -1.585 0.0075)
+			(end 1.585 0.0075)
+			(stroke
+				(width 0.1)
+				(type solid)
+			)
+			(layer "B.SilkS")
+		)
+		(fp_line
 			(start -1.585 -6.4025)
 			(end -0.94253 -6.4025)
@@
 			)
 			(layer "B.SilkS")
-		)
-		(fp_line
-			(start 0 -6.4025)
-			(end 0 6.4025)
-			(stroke
-				(width 0.1)
-				(type solid)
-			)
-			(layer "Dwgs.User")
-		)
-		(fp_line
-			(start -1.585 0.0075)
-			(end 1.585 0.0075)
-			(stroke
-				(width 0.1)
-				(type solid)
-			)
-			(layer "Dwgs.User")
 		)
 		(fp_line
@@
 		(model "${KICAD10_3DMODEL_DIR}/Connector_PinSocket_1.27mm.3dshapes/PinSocket_2x10_P1.27mm_Vertical.step"
 			(offset
-				(xyz 0.635 5.7225 0)
+				(xyz 0.645 5.85 0)
 			)
 			(scale
@@
 			)
 			(rotate
-				(xyz 0 0 0)
-			)
-		)
+				(xyz -0 -0 -0)
+			)
+		)

Commit message: [FIX] add 12V trace for expanders and generate gerber for all relays related boards
Other:
- board text added: "relay_module ui_board_v1.0.0"
Changed lines of the file:
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@@
 			(outputformat 1)
 			(mirror no)
-			(drillshape 1)
+			(drillshape 0)
 			(scaleselection 1)
-			(outputdirectory "")
+			(outputdirectory "gerber_ui_board/")
 		)
 	)
@@
 		(layer "Edge.Cuts")
 	)
+	(gr_text "relay_module\nui_board_v1.0.0"
+		(at 124.75 100 0)
+		(layer "B.SilkS")
+		(effects
+			(font
+				(size 1 1)
+				(thickness 0.1)
+			)
+			(justify left bottom mirror)
+		)
+	)
 	(segment
