File: tooling/kicad/templates/extension_module_two_rows_10cm_template/extension_module_two_rows_10cm_template.kicad_pcb (KiCad board)
At the start: 2 copper layers, 130 x 85 mm, 6 parts, among them J1 Conn_01x07_Socket, J2 Conn_01x07_Socket, SW1 SW_DIP_x03

Commit message: [ADD] two rows extention module
Parts:
- moved J2 30.0 mm to (177.0, 80.0)
Other:
- board size 130 x 85 mm -> 100 x 85 mm

Commit message: [ADD] board connector
Parts:
- moved J1 3.50 mm to (88.0, 83.5)
- moved J2 3.50 mm to (177.0, 83.5)
Changed lines of the file:
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@@
 		(locked yes)
 		(layer "F.Cu")
-		(at 177 80)
+		(at 177 83.5)
 		(descr "Through hole angled socket strip, 1x07, 2.54mm pitch, 8.51mm socket length, single row (from Kicad 4.0.7), script generated")
 		(tags "Through hole angled socket strip THT 1x07 2.54mm single row")
@@
 		(locked yes)
 		(layer "F.Cu")
-		(at 88 80)
+		(at 88 83.5)
 		(descr "Through hole angled pin header, 1x07, 2.54mm pitch, 6mm pin length, single row")
 		(tags "Through hole angled pin header THT 1x07 2.54mm single row")
